File: layouts/default/default.kicad_pcb (KiCad board)
At the start: 2 copper layers, 240 x 42 mm, 122 parts

Commit message: Add 6 M3 mounting holes (NPTH) and regenerate fab outputs
Parts:
- added H1: MountingHole_M3, , F.Cu at (53.0, 53.0)
- added H2: MountingHole_M3, , F.Cu at (53.0, 72.0)
- added H3: MountingHole_M3, , F.Cu at (177.0, 59.0)
- added H4: MountingHole_M3, , F.Cu at (172.4, 85.2)
- added H5: MountingHole_M3, , F.Cu at (287.0, 59.0)
- added H6: MountingHole_M3, , F.Cu at (287.0, 89.0)

Commit message: Move charge LEDs to bottom edge so bars don't cover them
The Gritin bars are ~40mm front-to-back centered on the plug (y=66),
covering everything up to y~86. LEDs moved from y=84 to y=91 (25mm
from plug center) with scripted B.Cu via-hop extensions under the
5V-B rail; DRC still clean, connectivity intact. Fab outputs
regenerated.
Parts:
- moved LED2 7.00 mm to (118.8, 91.0)
- moved LED3 7.00 mm to (141.2, 91.0)
- moved LED4 7.00 mm to (163.8, 91.0)
- moved LED5 7.00 mm to (186.2, 91.0)
- moved LED6 7.00 mm to (208.8, 91.0)
- moved LED7 7.00 mm to (231.2, 91.0)
- moved LED8 7.00 mm to (253.8, 91.0)
- moved LED9 7.00 mm to (276.2, 91.0)
Routing:
- net ports[3]-power_in-anode: track 259.5 -> 287.5 mm, vias 5 -> 13
- net ports[7]-power_in-anode: track 495.8 -> 523.8 mm, vias 24 -> 32
- net ports[4]-cathode: track 7.13 -> 14.1 mm, vias 0 -> 2
- net ports[1]-cathode: track 7.13 -> 14.1 mm, vias 0 -> 2
- net ports[7]-cathode: track 7.07 -> 14.1 mm, vias 0 -> 2
- net ports[6]-cathode: track 7.03 -> 14.0 mm, vias 0 -> 2
- net ports[5]-cathode: track 7.13 -> 14.1 mm, vias 0 -> 2
- net ports[3]-cathode: track 7.13 -> 14.1 mm, vias 0 -> 2
- net ports[0]-cathode: track 7.13 -> 14.1 mm, vias 0 -> 2
- net ports[2]-cathode: track 7.64 -> 14.6 mm, vias 0 -> 2

Commit message: Extend bottom edge 5mm (240x47) for LED visibility margin; move H4/H6 into new strip, add H7
Parts:
- added H7: MountingHole_M3, , F.Cu at (53.0, 94.0)
- moved H4 8.80 mm to (172.4, 94.0)
- moved H6 5.00 mm to (287.0, 94.0)
Other:
- board size 240 x 42 mm -> 240 x 47 mm
Changed lines of the file:
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@@
 	(footprint ""
 		(layer "F.Cu")
-		(at 172.4 85.2)
+		(at 172.4 94)
 		(property "Reference" "H4"
 			(at 0 0 0)
@@
 			(drill 3.2)
 			(layers "*.Cu" "*.Mask")
-			(clearance 0.4)
+			(clearance 0.5)
 		)
 		(embedded_fonts no)
@@
 	(footprint ""
 		(layer "F.Cu")
+		(at 53 94)
+		(property "Reference" "H7"
+			(at 0 0 0)
+			(layer "F.Fab")
+			(hide yes)
+			(effects
+				(font
+					(size 1.27 1.27)
+				)
+			)
+		)
+		(property "Value" "MountingHole_M3"
+			(at 0 0 0)
+			(layer "F.Fab")
+			(hide yes)
+			(effects
+				(font
+					(size 1.27 1.27)
+				)
+			)
+		)
+		(property "Datasheet" ""
+			(at 0 0 0)
+			(layer "F.Fab")
+			(hide yes)
+			(effects
+				(font
+					(size 1.27 1.27)
+				)
+			)
+		)
+		(property "Description" ""
+			(at 0 0 0)
+			(layer "F.Fab")
+			(hide yes)
+			(effects
+				(font
+					(size 1.27 1.27)
+				)
+			)
+		)
+		(attr board_only exclude_from_pos_files exclude_from_bom)
+		(duplicate_pad_numbers_are_jumpers no)
+		(pad "" np_thru_hole circle
+			(at 0 0)
+			(size 3.2 3.2)
+			(drill 3.2)
+			(layers "*.Cu" "*.Mask")
+			(clearance 0.5)
+		)
+		(embedded_fonts no)
+	)
+	(footprint ""
+		(layer "F.Cu")
 		(at 177 59)
 		(property "Reference" "H3"
@@
 	(footprint ""
 		(layer "F.Cu")
-		(at 287 89)
+		(at 287 94)
 		(property "Reference" "H6"
 			(at 0 0 0)
@@
 	)
 	(gr_line
-		(start 50 92)
+		(start 50 97)
 		(end 50 50)
 		(stroke
@@
 	(gr_line
 		(start 290 50)
-		(end 290 92)
+		(end 290 97)
 		(stroke
 			(width 0.1)
@@
 	)
 	(gr_line
-		(start 290 92)
-		(end 50 92)
+		(start 290 97)
+		(end 50 97)
 		(stroke
 			(width 0.1)
@@
 		(polygon
 			(pts
-				(xy 50.5 50.5) (xy 289.5 50.5) (xy 289.5 91.5) (xy 50.5 91.5)
+				(xy 50.5 50.5) (xy 289.5 50.5) (xy 289.5 96.5) (xy 50.5 96.5)
 			)
 		)
