File: ci/artifacts/v3-manufacturing.kicad_pcb (KiCad board)
At the start: 2 copper layers, 240 x 47 mm, 164 parts, among them SW1 TS-1187A-B-A-B, U1 INA3221AIRGVR, U10 74HC595, U11 74HC595, U12 HT7533-1, U2 INA3221AIRGVR, U3 TPS54560DDAR, U4 TPS54560DDAR, U5 CH224K, U6 INA3221AIRGVR, U7 CH32V203F6P6, U8 SN74HC4051DR, U9 SN74HC4051DR

Commit message: Fix lib_footprint_mismatch: update board FPs from libs
Syncing one resistor into the library reintroduced mismatches via
per-instance property angles. Make .pretty canonical (pad form, no
shell silk, no shared Supplier PN) and refresh all embeds from libs.

Co-authored-by: Cursor <cursoragent@cursor.com>
Connections:
- USB2 pad 14: (no net) -> port_0_vbus
- USB2 pad 15: port_0_vbus -> gnd
- USB2 pad 16: gnd -> (no net)
- USB2 pad 6: (no net) -> port_0_vbus
- USB2 pad 7: port_0_vbus -> gnd
- USB2 pad 8: gnd -> (no net)
- USB3 pad 14: (no net) -> port_1_vbus
- USB3 pad 15: port_1_vbus -> gnd
- USB3 pad 16: gnd -> (no net)
- USB3 pad 6: (no net) -> port_1_vbus
- USB3 pad 7: port_1_vbus -> gnd
- USB3 pad 8: gnd -> (no net)
- USB4 pad 14: (no net) -> port_2_vbus
- USB4 pad 15: port_2_vbus -> gnd
- USB4 pad 16: gnd -> (no net)
- USB4 pad 6: (no net) -> port_2_vbus
- USB4 pad 7: port_2_vbus -> gnd
- USB4 pad 8: gnd -> (no net)
- USB5 pad 14: (no net) -> port_3_vbus
- USB5 pad 15: port_3_vbus -> gnd
- USB5 pad 16: gnd -> (no net)
- USB5 pad 6: (no net) -> port_3_vbus
- USB5 pad 7: port_3_vbus -> gnd
- USB5 pad 8: gnd -> (no net)
- USB6 pad 14: (no net) -> port_4_vbus
- USB6 pad 15: port_4_vbus -> gnd
- USB6 pad 16: gnd -> (no net)
- USB6 pad 6: (no net) -> port_4_vbus
- USB6 pad 7: port_4_vbus -> gnd
- USB6 pad 8: gnd -> (no net)
- USB7 pad 14: (no net) -> port_5_vbus
- USB7 pad 15: port_5_vbus -> gnd
- USB7 pad 16: gnd -> (no net)
- USB7 pad 6: (no net) -> port_5_vbus
- USB7 pad 7: port_5_vbus -> gnd
- USB7 pad 8: gnd -> (no net)
- USB8 pad 14: (no net) -> port_6_vbus
- USB8 pad 15: port_6_vbus -> gnd
- USB8 pad 16: gnd -> (no net)
- USB8 pad 6: (no net) -> port_6_vbus
- USB8 pad 7: port_6_vbus -> gnd
- USB8 pad 8: gnd -> (no net)
- USB9 pad 14: (no net) -> port_7_vbus
- USB9 pad 15: port_7_vbus -> gnd
- USB9 pad 16: gnd -> (no net)
- USB9 pad 6: (no net) -> port_7_vbus
- USB9 pad 7: port_7_vbus -> gnd
- USB9 pad 8: gnd -> (no net)

Commit message: Restore copper; clear lib mismatch via property-at normalize
Revert board FP rewrite that broke nets/shorts. Keep silk/PN hygiene,
align shared .pretty pad/silk form, strip property (at) angles that
differ per rotation, and stop using update-board-fps-from-lib by default.

Co-authored-by: Cursor <cursoragent@cursor.com>
Connections:
- USB2 pad 14: port_0_vbus -> (no net)
- USB2 pad 15: gnd -> port_0_vbus
- USB2 pad 16: (no net) -> gnd
- USB2 pad 6: port_0_vbus -> (no net)
- USB2 pad 7: gnd -> port_0_vbus
- USB2 pad 8: (no net) -> gnd
- USB3 pad 14: port_1_vbus -> (no net)
- USB3 pad 15: gnd -> port_1_vbus
- USB3 pad 16: (no net) -> gnd
- USB3 pad 6: port_1_vbus -> (no net)
- USB3 pad 7: gnd -> port_1_vbus
- USB3 pad 8: (no net) -> gnd
- USB4 pad 14: port_2_vbus -> (no net)
- USB4 pad 15: gnd -> port_2_vbus
- USB4 pad 16: (no net) -> gnd
- USB4 pad 6: port_2_vbus -> (no net)
- USB4 pad 7: gnd -> port_2_vbus
- USB4 pad 8: (no net) -> gnd
- USB5 pad 14: port_3_vbus -> (no net)
- USB5 pad 15: gnd -> port_3_vbus
- USB5 pad 16: (no net) -> gnd
- USB5 pad 6: port_3_vbus -> (no net)
- USB5 pad 7: gnd -> port_3_vbus
- USB5 pad 8: (no net) -> gnd
- USB6 pad 14: port_4_vbus -> (no net)
- USB6 pad 15: gnd -> port_4_vbus
- USB6 pad 16: (no net) -> gnd
- USB6 pad 6: port_4_vbus -> (no net)
- USB6 pad 7: gnd -> port_4_vbus
- USB6 pad 8: (no net) -> gnd
- USB7 pad 14: port_5_vbus -> (no net)
- USB7 pad 15: gnd -> port_5_vbus
- USB7 pad 16: (no net) -> gnd
- USB7 pad 6: port_5_vbus -> (no net)
- USB7 pad 7: gnd -> port_5_vbus
- USB7 pad 8: (no net) -> gnd
- USB8 pad 14: port_6_vbus -> (no net)
- USB8 pad 15: gnd -> port_6_vbus
- USB8 pad 16: (no net) -> gnd
- USB8 pad 6: port_6_vbus -> (no net)
- USB8 pad 7: gnd -> port_6_vbus
- USB8 pad 8: (no net) -> gnd
- USB9 pad 14: port_7_vbus -> (no net)
- USB9 pad 15: gnd -> port_7_vbus
- USB9 pad 16: (no net) -> gnd
- USB9 pad 6: port_7_vbus -> (no net)
- USB9 pad 7: gnd -> port_7_vbus
- USB9 pad 8: (no net) -> gnd
