File: ci/artifacts/v3-for-route.kicad_pcb (KiCad board)
At the start: 2 copper layers, 240 x 47 mm, 164 parts, among them SW1 TS-1187A-B-A-B, U1 INA3221AIRGVR, U10 74HC595, U11 74HC595, U12 HT7533-1, U2 INA3221AIRGVR, U3 TPS54560DDAR, U4 TPS54560DDAR, U5 CH224K, U6 INA3221AIRGVR, U7 CH32V203F6P6, U8 SN74HC4051DR, U9 SN74HC4051DR

Commit message: Update V3 board renders
Parts:
- R10, R6: value 17.8kΩ -> 17.8kÎ©
- R11, R7: value 3.4kΩ -> 3.4kÎ©
- R12, R8: value 162kΩ -> 162kÎ©
- R13, R14, R17: value 24kΩ -> 24kÎ©
- R15, R16, R77: value 100kΩ -> 100kÎ©
- R18, R69, R70: value 4.7kΩ -> 4.7kÎ©
- R19, R53, R54, R55, R56, R57, R58, R59, R60, R61, R62, R63, R64, R65, R66, R67, R68, R72: value 1kΩ -> 1kÎ©
- R20, R21, R24, R25, R28, R29, R32, R33, R36, R37, R40, R41, R44, R45, R48, R49: value 22kΩ -> 22kÎ©
- R23, R27, R31, R35, R39, R43, R47, R51: value 100mΩ -> 100mÎ©
- R5, R9: value 23.7kΩ -> 23.7kÎ©
- R52, R71, R73, R74, R75, R76: value 10kΩ -> 10kÎ©
- moved SW1 101.8 mm to (10.0, 121.8)
- renumbered REF3 to ?, REF2 to ?, REF10 to ?, REF8 to ?, REF1 to ?, REF5 to ?, REF7 to ?, REF9 to ?, REF4 to ?, REF6 to ?
Other:
- board text added: "IN: USB C PD 12V OR DC 12V"
- board text added: "OUT: 5V 1A/PORT"
- board text added: "SKG // LIGHTBAR DOCK // V3"
